File: Test/Test.kicad_pcb (KiCad board)
At the start: 2 copper layers, 53.3 x 45.7 mm, 10 parts, among them J1 DIN-6, J2 DIN-6, SW1 SW_Push, SW2 SW_Push, SW3 SW_Push, SW4 SW_Push, SW5 SW_Push, SW6 SW_Push, U1 ProMicro

Commit message: Initial Gerber (not tested)
Parts:
- removed SW1, SW2, SW3, SW4, SW5, SW6: SW_Push, Button_Switch_THT:SW_PUSH_6mm_H5mm
- added DCAL1: LED_Filled, LED_THT:LED_D5.0mm_FlatTop, F.Cu at (116.8, 73.7)
- added DLEFT1: LED_Filled, LED_THT:LED_D5.0mm_FlatTop, F.Cu at (147.3, 73.7)
- added DRIGHT1: LED_Filled, LED_THT:LED_D5.0mm_FlatTop, F.Cu at (73.7, 73.7)
- added R1: R, Resistor_THT:R_Axial_DIN0207_L6.3mm_D2.5mm_P10.16mm_Horizontal, F.Cu at (73.7, 81.3)
- added R2: R, Resistor_THT:R_Axial_DIN0207_L6.3mm_D2.5mm_P10.16mm_Horizontal, F.Cu at (147.3, 78.7)
- added R3: R, Resistor_THT:R_Axial_DIN0207_L6.3mm_D2.5mm_P10.16mm_Horizontal, F.Cu at (120.7, 78.7)
- added SWCAL1: SW_Push, Connector_PinSocket_2.54mm:PinSocket_1x02_P2.54mm_Vertical, F.Cu at (105.4, 76.2)
- added SWPROG1: SW_SPDT, Connector_PinSocket_2.54mm:PinSocket_1x03_P2.54mm_Vertical, F.Cu at (135.9, 95.2)
- added SWREPEAT1: SW_Push, Connector_PinSocket_2.54mm:PinSocket_1x02_P2.54mm_Vertical, F.Cu at (128.3, 95.2)
- moved SW_RST1 35.9 mm to (91.4, 99.1), turned to 180 degrees
- moved JLEFT1 35.8 mm to (132.1, 80.0)
- moved JRIGHT1 34.7 mm to (91.4, 80.0)
- moved U1 32.1 mm to (111.8, 99.1), turned to 90 degrees
- renumbered J2 to JLEFT1, J1 to JRIGHT1
Connections:
- net Axis X 2 renamed Axis X R
- net Axis Y 2 renamed Axis Y R
- net BLACK 2 renamed BLACK R
- JLEFT1 pad 1: Axis X 1 -> Axis X L
- JLEFT1 pad 2: Axis Y 1 -> Axis Y L
- JLEFT1 pad 4: RED 1 -> RED L
- JLEFT1 pad 6: BLACK 1 -> BLACK L
- JRIGHT1 pad 4: RED 2 -> RED R
- U1 pad 10: Net-(SW3-Pad1) -> RED L
- U1 pad 11: Net-(SW2-Pad1) -> BLACK L
- U1 pad 12: Net-(SW1-Pad1) -> DCAL
- U1 pad 14: BLACK 1 -> RED R
- U1 pad 15: RED 2 -> DRIGHT
- U1 pad 16: RED 1 -> SWCAL
- U1 pad 17: Axis Y 1 -> Axis X L
- U1 pad 18: Axis X 1 -> Axis Y L
- U1 pad 6: unconnected-(U1-Pad6) -> SWPROG
- U1 pad 7: Net-(SW6-Pad1) -> SWREPEAT
- U1 pad 8: Net-(SW5-Pad1) -> unconnected-(U1-Pad8)
- U1 pad 9: Net-(SW4-Pad1) -> DLEFT
Routing:
- net 5V: track 54.7 -> 120.2 mm, vias 0 -> 2
- net GND: track 262.3 -> 207.3 mm, vias 1 -> 0
- net DRIGHT: track 0.00 -> 44.0 mm, vias 0 -> 2
- net DLEFT: track 0.00 -> 42.1 mm
- net RED 1: track 36.8 -> 0.00 mm
- net BLACK 1: track 32.3 -> 0.00 mm
- net Net-(SW4-Pad1): track 28.4 -> 0.00 mm
- net BLACK R: track 41.8 -> 13.6 mm
- net Axis Y L: track 0.00 -> 28.0 mm
- net Net-(SW5-Pad1): track 28.0 -> 0.00 mm
- net Net-(SW3-Pad1): track 25.6 -> 0.00 mm
- net Axis X L: track 0.00 -> 25.5 mm
- net SWCAL: track 0.00 -> 23.0 mm, vias 0 -> 2
- net SWPROG: track 0.00 -> 21.2 mm
- net RED L: track 0.00 -> 19.6 mm
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Other:
- board size 53.3 x 45.7 mm -> 83.8 x 44.5 mm
