File: Test/Test.kicad_sch (KiCad schematic)
At the start: 10 parts, among them U1 ProMicro

Commit message: Initial Gerber (not tested)
Parts:
- removed SW1, SW2, SW3, SW4, SW5, SW6: (no value), symbol Switch:SW_Push
- added DCAL1, DRIGHT1: (no value), symbol Device:LED_Filled
- added DLEFT1: LED_Filled, symbol Device:LED_Filled
- added R1: (no value), symbol Device:R
- added R2: R, symbol Device:R
- added R3: R, Resistor_THT:R_Axial_DIN0207_L6.3mm_D2.5mm_P10.16mm_Horizontal, symbol Device:R
- added SWCAL1, SWREPEAT1: (no value), symbol Switch:SW_Push
- added SWPROG1: (no value), symbol Switch:SW_SPDT
- JLEFT1: renamed from J2; value (none) -> DIN-6; footprint (none) -> Connectors_UNITRA:DIN-6
- JRIGHT1: renamed from J1; value (none) -> DIN-6; footprint (none) -> Connectors_UNITRA:DIN-6
- U1: footprint (none) -> promicro:ProMicro
Connections:
- net 5V: now also SWPROG1.3 (C)
- net GND: now also R1.2, R2.2, R3.2, SWCAL1.1, SWPROG1.1 (A), SWREPEAT1.1
- net RED L: now reaches U1.10 (E6)
- net RED L: now also JLEFT1.4
- net DCAL: now reaches U1.12 (B5)
- net DCAL: now also DCAL1.2 (A)
- net BLACK L: now reaches U1.11 (B4)
- net BLACK L: now also JLEFT1.6
- net SWREPEAT: now reaches U1.7 (D4)
- net SWREPEAT: now also SWREPEAT1.2
- net DLEFT: now reaches U1.9 (D7)
- net DLEFT: now also DLEFT1.2 (A)
- net SWPROG: now reaches U1.6 (SCL)
- net SWPROG: now also SWPROG1.2 (B)
- net Axis X 1 renamed Axis X L
- net Axis X L: now also U1.17 (F7); no longer U1.18 (F6)
- net Axis X 2 renamed Axis X R
- net Axis Y 1 renamed Axis Y L
- net Axis Y L: now also U1.18 (F6); no longer U1.17 (F7)
- net Axis Y 2 renamed Axis Y R
- net BLACK 1 renamed RED R
- net RED R: now also JRIGHT1.4; no longer JLEFT1.6
- net BLACK 2 renamed BLACK R
- net RED 1 renamed SWCAL
- net SWCAL: now also SWCAL1.2; no longer JLEFT1.4
- net RED 2 renamed DRIGHT
- net DRIGHT: now also DRIGHT1.2 (A); no longer JRIGHT1.4
- new net: DRIGHT1.1 (K), R1.1
- new net: DCAL1.1 (K), R3.1
- new net: DLEFT1.1 (K), R2.1
- no-connect marks 5 -> 3
